Commit message: modified launch, rviz-config and ros2_control params files

File: robot_desc/ros2_control.xacro (robot description, xacro)
@@ -42,4 +42,12 @@
         <state_interface name="velocity"/>
       </joint>
+      <joint name="camera_joint">
+        <command_interface name="position">
+          <param name="min">-0.785</param>
+          <param name="max">0.785</param>
+        </command_interface>
+        <state_interface name="position"/>
+        <state_interface name="velocity"/>
+      </joint>
     </ros2_control>
 </robot>
